File: Hardware/RP2040 Module.kicad_pcb (KiCad board)
At the start: 4 copper layers, 66 x 24.1 mm, 14 parts, among them J1 Conn_01x09, J2 Conn_01x09, J3 Conn_01x09, J4 Conn_01x09, U1 ADuM1201AR, U2 RP2040, U3 HT7533, U4 W25Q32JVSS, Y1 12MHz

Commit message: updated files
Parts:
- removed J1, J2, J3, J4: Conn_01x09, Connector_PinHeader_1.27mm:PinHeader_1x09_P1.27mm_Vertical
- removed U4: W25Q32JVSS, Package_SO:SOIC-8_5.23x5.23mm_P1.27mm
- added C10: 10uF, Capacitor_SMD:C_0402_1005Metric, F.Cu at (152.5, 105.5)
- added C11: 10uF, Capacitor_SMD:C_0402_1005Metric, F.Cu at (150.3, 94.7)
- added C12: 10uF, Capacitor_SMD:C_0402_1005Metric, F.Cu at (144.8, 97.4)
- added C13: 10uF, Capacitor_SMD:C_0402_1005Metric, F.Cu at (153.0, 94.7)
- added C6: 10uF, Capacitor_SMD:C_0402_1005Metric, F.Cu at (153.4, 105.5)
- added C7: 10uF, Capacitor_SMD:C_0402_1005Metric, F.Cu at (152.1, 94.7)
- added C8: 10uF, Capacitor_SMD:C_0402_1005Metric, F.Cu at (149.4, 94.7)
- added C9: 10uF, Capacitor_SMD:C_0402_1005Metric, F.Cu at (155.2, 97.4)
- added R1: 1K, Resistor_SMD:R_0402_1005Metric, F.Cu at (176.0, 94.8)
- added R2: 10K, Resistor_SMD:R_0402_1005Metric, F.Cu at (173.1, 96.7)
- added R3: 10K, Resistor_SMD:R_0402_1005Metric, F.Cu at (173.1, 94.8)
- added R4: 22R, Resistor_SMD:R_0402_1005Metric, F.Cu at (152.1, 92.4)
- added R5: 27R, Resistor_SMD:R_0402_1005Metric, F.Cu at (150.3, 92.4)
- added SW1: RST, Button_Switch_SMD:SW_SPST_B3U-1000P, F.Cu at (159.0, 90.0)
- added SW2: BOOTSEL, Button_Switch_SMD:SW_SPST_B3U-1000P, F.Cu at (159.0, 93.0)
- added U6: W25Q64JVXGIQ_TR, 25Q64:W25Q64JVXGIQ TR, F.Cu at (144.6, 92.1)
- moved C4 28.6 mm to (179.6, 108.5), turned to -90 degrees
- moved U3 27.9 mm to (176.1, 107.5), turned to 180 degrees
- moved C5 26.7 mm to (146.1, 89.3), turned to 180 degrees
- moved U1 24.8 mm to (129.2, 101.5)
- moved C3 21.9 mm to (172.6, 108.5), turned to 90 degrees
- moved U2 20.9 mm to (150.0, 100.0)
- moved Y1 17.7 mm to (149.1, 106.1)
- moved C1 16.6 mm to (151.6, 105.5), turned to -90 degrees
- moved C2 11.7 mm to (146.6, 105.5), turned to -90 degrees
Connections:
- net Net-(C3-Pad2) renamed VCC
- C1 pad 1: Net-(C1-Pad1) -> Net-(U2-Pad21)
- C2 pad 2: Net-(Y1-Pad1) -> Net-(U2-Pad20)
- C4 pad 1: +3.3V -> +3V3
- C5 pad 1: GND -> +3V3
- C5 pad 2: +3.3V -> GND
- U1 pad 1: unconnected-(U1-Pad1) -> +3V3
- U1 pad 4: unconnected-(U1-Pad4) -> GND
- U1 pad 5: unconnected-(U1-Pad5) -> /ISO_GND
- U1 pad 6: unconnected-(U1-Pad6) -> /ISO_VO
- U1 pad 7: unconnected-(U1-Pad7) -> /ISO_VIN
- U1 pad 8: unconnected-(U1-Pad8) -> /ISO_VCC
- U2 pad 1: Net-(U2-Pad1) -> +3V3
- U2 pad 10: Net-(U2-Pad1) -> +3V3
- U2 pad 11: unconnected-(U2-Pad11) -> /GPIO8
- U2 pad 12: unconnected-(U2-Pad12) -> /GPIO9
- U2 pad 13: unconnected-(U2-Pad13) -> /GPIO10
- U2 pad 14: unconnected-(U2-Pad14) -> /GPIO11
- U2 pad 15: unconnected-(U2-Pad15) -> /GPIO12
- U2 pad 16: unconnected-(U2-Pad16) -> /GPIO13
- U2 pad 17: unconnected-(U2-Pad17) -> /GPIO14
- U2 pad 18: unconnected-(U2-Pad18) -> /GPIO15
- U2 pad 19: unconnected-(U2-Pad19) -> GND
- U2 pad 2: unconnected-(U2-Pad2) -> /GPIO0
- U2 pad 20: unconnected-(U2-Pad20) -> Net-(U2-Pad20)
- U2 pad 21: unconnected-(U2-Pad21) -> Net-(U2-Pad21)
- U2 pad 22: Net-(U2-Pad1) -> +3V3
- U2 pad 23: Net-(U2-Pad23) -> +1V1
- U2 pad 26: unconnected-(U2-Pad26) -> /RST
- U2 pad 27: unconnected-(U2-Pad27) -> /GPIO16
- U2 pad 28: unconnected-(U2-Pad28) -> /GPIO17
- U2 pad 29: unconnected-(U2-Pad29) -> /GPIO18
- U2 pad 3: unconnected-(U2-Pad3) -> /GPIO1
- U2 pad 30: unconnected-(U2-Pad30) -> /GPIO19
- U2 pad 31: unconnected-(U2-Pad31) -> /GPIO20
- U2 pad 32: unconnected-(U2-Pad32) -> /GPIO21
- U2 pad 33: Net-(U2-Pad1) -> +3V3
- U2 pad 34: unconnected-(U2-Pad34) -> /GPIO22
- U2 pad 35: unconnected-(U2-Pad35) -> /GPIO23
- U2 pad 36: unconnected-(U2-Pad36) -> /GPIO24
- U2 pad 37: unconnected-(U2-Pad37) -> /GPIO25
- U2 pad 38: unconnected-(U2-Pad38) -> /GPIO26
- U2 pad 39: unconnected-(U2-Pad39) -> /GPIO27
- U2 pad 4: unconnected-(U2-Pad4) -> /GPIO2
- U2 pad 40: unconnected-(U2-Pad40) -> /GPIO28
- U2 pad 41: unconnected-(U2-Pad41) -> /GPIO29
- U2 pad 42: Net-(U2-Pad1) -> +3V3
- U2 pad 43: unconnected-(U2-Pad43) -> +3V3
- U2 pad 44: unconnected-(U2-Pad44) -> +3V3
- U2 pad 45: unconnected-(U2-Pad45) -> +1V1
- U2 pad 46: unconnected-(U2-Pad46) -> Net-(U2-Pad46)
- U2 pad 47: unconnected-(U2-Pad47) -> Net-(U2-Pad47)
- U2 pad 48: unconnected-(U2-Pad48) -> +3V3
- U2 pad 49: Net-(U2-Pad1) -> +3V3
- U2 pad 5: unconnected-(U2-Pad5) -> /GPIO3
- U2 pad 50: Net-(U2-Pad23) -> +1V1
- U2 pad 57: unconnected-(U2-Pad57) -> GND
- U2 pad 6: unconnected-(U2-Pad6) -> /GPIO4
- U2 pad 7: unconnected-(U2-Pad7) -> /GPIO5
- U2 pad 8: unconnected-(U2-Pad8) -> /GPIO6
- U2 pad 9: unconnected-(U2-Pad9) -> /GPIO7
- U3 pad 3: +3.3V -> +3V3
- Y1 pad 1: Net-(Y1-Pad1) -> Net-(U2-Pad20)
- Y1 pad 3: Net-(C1-Pad1) -> Net-(U2-Pad21)
Routing:
- net Net-(U2-Pad47): track 0.00 -> 3.85 mm
- net Net-(U2-Pad46): track 0.00 -> 3.85 mm
- net GND: vias 0 -> 7
- added copper zone on F.Cu, net +1V1
- added copper zone on F.Cu, net +3V3
- added copper zone on F.Cu, net GND
Other:
- board size 66 x 24.1 mm -> 25 x 25 mm

Commit message: updated files
Parts:
- added J1: IO, Connector_PinHeader_2.00mm:PinHeader_1x10_P2.00mm_Vertical, F.Cu at (141.0, 87.5)
- added J2: IO, Connector_PinHeader_2.00mm:PinHeader_1x10_P2.00mm_Vertical, F.Cu at (162.5, 91.0)
- added J3: IO, Connector_PinHeader_2.00mm:PinHeader_1x10_P2.00mm_Vertical, F.Cu at (159.0, 112.5)
- added J4: IO, Connector_PinHeader_2.00mm:PinHeader_1x10_P2.00mm_Vertical, F.Cu at (137.5, 109.0)
- moved R1 33.0 mm to (143.0, 93.5)
- moved C4 32.7 mm to (146.9, 108.0)
- moved U3 32.4 mm to (143.7, 107.0)
- moved R2 32.3 mm to (141.0, 93.5)
- moved C3 32.1 mm to (140.5, 108.0)
- moved U1 28.7 mm to (156.6, 92.7)
- moved R3 19.9 mm to (157.0, 106.5)
- moved SW1 18.7 mm to (158.0, 108.7), turned to 180 degrees
- moved SW2 17.1 mm to (142.0, 91.3)
- moved U6 8.32 mm to (142.0, 100.0), turned to 90 degrees
- moved C9 7.47 mm to (151.7, 90.8)
- moved C5 6.01 mm to (150.5, 93.4), turned to 90 degrees
- moved C11 5.70 mm to (144.6, 94.9), turned to 0 degrees
- moved C8 4.92 mm to (144.6, 95.8), turned to 0 degrees
- moved C2 4.91 mm to (151.1, 107.4), turned to -45 degrees
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Connections:
- R3 pad 1: Net-(R1-Pad1) -> +3V3
Routing:
- net +3V3: track 0.00 -> 16.6 mm
- net /IO2: track 0.00 -> 10.3 mm, vias 0 -> 2
- net /IO1: track 0.00 -> 10.1 mm, vias 0 -> 2
- net +1V1: track 0.00 -> 9.13 mm
- net /~{CS}: track 0.00 -> 8.37 mm, vias 0 -> 2
- net /IO3: track 0.00 -> 7.25 mm
- net Net-(C2-Pad2): track 0.00 -> 6.79 mm
- net /CLK: track 0.00 -> 5.95 mm
- net /IO0: track 0.00 -> 4.66 mm
- net Net-(C1-Pad1): track 0.00 -> 4.01 mm
- net /GPIO0: track 0.00 -> 1.29 mm, vias 0 -> 1
- net /GPIO6: track 0.00 -> 1.29 mm, vias 0 -> 1
- net /GPIO9: track 0.00 -> 1.27 mm, vias 0 -> 1
- net /GPIO4: track 0.00 -> 1.26 mm, vias 0 -> 1
- net /GPIO2: track 0.00 -> 1.24 mm, vias 0 -> 1
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- added copper zone on B.Cu, net GND
- added copper zone on In1.Cu, net GND
- added copper zone on F.Cu, net VCC
- removed copper zone on F.Cu, net +1V1
Other:
- outline, holes or cut-outs redrawn

Commit message: updated files
Parts:
- added kibuzzard-63D05A78: G***, kibuzzard-63D05A78, F.Cu at (157.2, 96.8)
- moved C1 4.53 mm to (154.8, 108.7), turned to -90 degrees
- moved Y1 2.94 mm to (152.5, 108.7), turned to 0 degrees
- moved C2 1.58 mm to (150.2, 108.7), turned to -90 degrees
- moved C4 1.00 mm to (145.9, 108.0)
- moved C10 0.81 mm to (155.7, 103.9), turned to 180 degrees
- moved U3 0.70 mm to (143.0, 107.0)
- moved C6 0.64 mm to (156.2, 102.4), turned to 180 degrees
- moved C3 0.40 mm to (140.1, 108.0)
- moved R1 0.19 mm to (143.2, 93.5)
- moved R2 0.19 mm to (140.8, 93.5)
- moved C12 0.10 mm to (140.7, 96.6)
- moved U6 0.10 mm to (141.9, 100.0)
Routing:
- net GND: track 0.52 -> 5.91 mm, vias 1 -> 6
- net /~{CS}: track 8.37 -> 13.1 mm, vias 2 -> 0
- net Net-(C1-Pad1): track 4.01 -> 7.23 mm
- net +1V1: track 9.13 -> 6.15 mm
- net /GPIO7: track 0.73 -> 3.26 mm
- net /GPIO8: track 0.81 -> 3.11 mm
- net +3V3: track 16.6 -> 18.8 mm
- net /GPIO29: track 0.00 -> 2.10 mm, vias 0 -> 1
- net /GPIO6: track 1.29 -> 3.29 mm
- net Net-(C2-Pad2): track 6.79 -> 8.65 mm
- net /GPIO9: track 1.27 -> 3.14 mm
- net /GPIO10: track 0.73 -> 2.36 mm
- net /GPIO5: track 0.89 -> 2.51 mm
- net /GPIO27: track 0.00 -> 1.44 mm, vias 0 -> 1
- net Net-(R1-Pad1): track 0.00 -> 1.36 mm
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
Commit message: updated files
Parts:
- removed kibuzzard-63D05A78: G***, kibuzzard-63D05A78
- moved C10 12.2 mm to (167.7, 101.6)
- moved C6 11.6 mm to (167.7, 100.6)
- moved Y1 4.98 mm to (155.0, 104.4), turned to -135 degrees
- moved R1 2.69 mm to (143.2, 90.8), turned to 90 degrees
- moved R3 2.48 mm to (158.9, 104.9)
- moved R2 2.41 mm to (143.2, 93.2), turned to 90 degrees
- moved U1 1.75 mm to (158.1, 93.6), turned to 90 degrees
- moved SW2 1.22 mm to (141.0, 92.0), turned to 90 degrees
- moved C1 0.63 mm to (154.2, 108.9)
- moved C2 0.63 mm to (149.6, 108.9)
Connections:
- U2 pad 24: unconnected-(U2-Pad24) -> /SWCLK
- U2 pad 25: unconnected-(U2-Pad25) -> /SWD
Routing:
- net Net-(C2-Pad2): track 8.65 -> 0.00 mm
- net Net-(C1-Pad1): track 7.23 -> 0.00 mm
- net /GPIO22: track 0.00 -> 4.10 mm, vias 0 -> 1
- net /GPIO24: track 0.00 -> 3.35 mm, vias 0 -> 1
- net /GPIO23: track 0.00 -> 3.33 mm, vias 0 -> 1
- net /GPIO14: track 0.00 -> 2.80 mm, vias 0 -> 1
- net GND: track 5.91 -> 3.12 mm
- net /GPIO15: track 0.00 -> 2.78 mm, vias 0 -> 1
- net /GPIO26: track 0.00 -> 2.61 mm, vias 0 -> 1
- net /GPIO25: track 0.00 -> 2.58 mm, vias 0 -> 1
- net /GPIO20: track 0.00 -> 2.09 mm, vias 0 -> 1
- net /GPIO21: track 0.00 -> 2.06 mm, vias 0 -> 1
- net /GPIO12: track 0.00 -> 2.06 mm, vias 0 -> 1
- net /GPIO13: track 0.00 -> 2.03 mm, vias 0 -> 1
- net /GPIO18: track 0.00 -> 1.34 mm, vias 0 -> 1
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
Commit message: updated files
Parts:
- moved C10 12.5 mm to (155.4, 104.0)
- moved C6 12.5 mm to (155.4, 103.0)
- moved Y1 4.19 mm to (153.2, 108.2), turned to 0 degrees
- moved R3 3.91 mm to (156.8, 108.2), turned to -90 degrees
- moved C9 2.61 mm to (151.5, 93.4), turned to -90 degrees
- moved C1 1.66 mm to (155.7, 108.2)
- moved SW1 1.56 mm to (159.0, 107.5), turned to -90 degrees
- moved C2 1.30 mm to (150.7, 108.2)
- moved R1 0.69 mm to (143.2, 91.5)
- moved SW2 0.50 mm to (141.0, 92.5)
- moved R2 0.31 mm to (143.2, 93.5)
- moved U1 0.22 mm to (158.0, 93.8)
Connections:
- J3 pad 1: unconnected-(J3-Pad1) -> /RST
- J3 pad 10: unconnected-(J3-Pad10) -> /GPIO8
- J3 pad 2: unconnected-(J3-Pad2) -> GND
- J3 pad 3: unconnected-(J3-Pad3) -> /GPIO15
- J3 pad 4: unconnected-(J3-Pad4) -> /GPIO14
- J3 pad 5: unconnected-(J3-Pad5) -> /GPIO13
- J3 pad 6: unconnected-(J3-Pad6) -> /GPIO12
- J3 pad 7: unconnected-(J3-Pad7) -> /GPIO11
- J3 pad 8: unconnected-(J3-Pad8) -> /GPIO10
- J3 pad 9: unconnected-(J3-Pad9) -> /GPIO9
- J4 pad 10: unconnected-(J4-Pad10) -> /GPIO0
- J4 pad 3: unconnected-(J4-Pad3) -> /GPIO7
- J4 pad 4: unconnected-(J4-Pad4) -> /GPIO6
- J4 pad 5: unconnected-(J4-Pad5) -> /GPIO5
- J4 pad 6: unconnected-(J4-Pad6) -> /GPIO4
- J4 pad 7: unconnected-(J4-Pad7) -> /GPIO3
- J4 pad 8: unconnected-(J4-Pad8) -> /GPIO2
- J4 pad 9: unconnected-(J4-Pad9) -> /GPIO1
- U1 pad 2: unconnected-(U1-Pad2) -> /GPIO19
- U1 pad 3: unconnected-(U1-Pad3) -> /GPIO18
Routing:
- net /GPIO0: track 1.05 -> 15.8 mm
- net /GPIO1: track 1.02 -> 14.9 mm
- net /GPIO2: track 1.79 -> 13.9 mm
- net /GPIO8: track 2.78 -> 14.3 mm
- net /GPIO3: track 1.77 -> 11.7 mm
- net /GPIO9: track 2.80 -> 12.5 mm
- net /GPIO4: track 2.54 -> 11.8 mm
- net /GPIO5: track 2.51 -> 11.5 mm
- net /GPIO7: track 3.26 -> 11.3 mm
- net /GPIO6: track 3.29 -> 11.3 mm
- net /GPIO15: track 2.78 -> 10.5 mm
- net /GPIO10: track 2.03 -> 9.61 mm
- net /GPIO11: track 2.06 -> 9.13 mm
- net Net-(C2-Pad2): track 0.00 -> 7.02 mm
- net /GPIO12: track 2.06 -> 9.05 mm
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
Commit message: updated files
Parts:
- moved U1 6.20 mm to (158.0, 100.0)
- moved C6 2.31 mm to (155.2, 105.3), turned to 90 degrees
- moved C10 1.77 mm to (154.2, 105.3), turned to 90 degrees
- moved R1 0.19 mm to (143.2, 91.3)
Connections:
- J1 pad 1: unconnected-(J1-Pad1) -> /~{CS}
- J1 pad 2: unconnected-(J1-Pad2) -> /GPIO29
- J1 pad 3: unconnected-(J1-Pad3) -> /GPIO28
- J1 pad 4: unconnected-(J1-Pad4) -> /GPIO27
- J1 pad 5: unconnected-(J1-Pad5) -> /GPIO26
- J1 pad 6: unconnected-(J1-Pad6) -> /GPIO25
- J1 pad 7: unconnected-(J1-Pad7) -> /GPIO24
- J1 pad 8: unconnected-(J1-Pad8) -> /GPIO23
- J1 pad 9: unconnected-(J1-Pad9) -> /GPIO22
- J2 pad 1: unconnected-(J2-Pad1) -> /ISO_VCC
- J2 pad 2: unconnected-(J2-Pad2) -> /ISO_VIN
- J2 pad 3: unconnected-(J2-Pad3) -> /ISO_VO
- J2 pad 4: unconnected-(J2-Pad4) -> /ISO_GND
Routing:
- net /GPIO29: track 1.09 -> 15.2 mm
- net /GPIO28: track 1.86 -> 14.2 mm
- net /GPIO27: track 1.92 -> 13.8 mm
- net /ISO_VCC: track 0.00 -> 10.4 mm
- net /GPIO26: track 2.61 -> 12.3 mm
- net /GPIO25: track 2.58 -> 11.6 mm
- net /GPIO22: track 4.10 -> 12.1 mm
- net /ISO_VIN: track 0.00 -> 7.92 mm
- net /GPIO23: track 3.33 -> 11.1 mm
- net /GPIO24: track 3.35 -> 10.8 mm
- net /~{CS}: track 10.9 -> 16.7 mm, vias 0 -> 1
- net /ISO_VO: track 0.00 -> 5.51 mm
- net /GPIO18: track 6.65 -> 1.69 mm
- net /GPIO19: track 5.53 -> 1.66 mm
- net /ISO_GND: track 0.00 -> 3.24 mm
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