File: Hardware/RP2040 Module.kicad_sch (KiCad schematic)
At the start: 3 parts

Commit message: updated files
Parts:
- removed U?: RP2040, Package_DFN_QFN:QFN-56-1EP_7x7mm_P0.4mm_EP3.2x3.2mm, symbol MCU_RaspberryPi:RP2040
- removed U?: W25Q16, Package_SO:SOIC-8_5.23x5.23mm_P1.27mm, symbol Memory_Flash:W25Q128JVS
- removed Y?: Crystal_GND24, symbol Device:Crystal_GND24
- added C1, C2: 22pF, Capacitor_SMD:C_0402_1005Metric, symbol Device:C_Small
- added C3, C4, C5: 10uF, Capacitor_SMD:C_0402_1005Metric, symbol Device:C_Small
- added J1, J2, J3, J4: Conn_01x09, Connector_PinHeader_1.27mm:PinHeader_1x09_P1.27mm_Vertical, symbol Connector_Generic:Conn_01x09
- added U1: ADuM1201AR, Package_SO:SOIC-8_3.9x4.9mm_P1.27mm, symbol Isolator:ADuM1201AR
- added U2: RP2040, Package_DFN_QFN:QFN-56-1EP_7x7mm_P0.4mm_EP3.2x3.2mm, symbol MCU_RaspberryPi:RP2040
- added U3: HT7533, Package_TO_SOT_SMD:SOT-89-3, symbol Regulator_Linear:HT75xx-1-SOT89
- added U4: W25Q32JVSS, Package_SO:SOIC-8_5.23x5.23mm_P1.27mm, symbol Memory_Flash:W25Q32JVSS
- added Y1: 12MHz, Oscillator:Oscillator_SMD_Abracon_ASE-4Pin_3.2x2.5mm, symbol Device:Crystal_GND24
Connections:
- new net: C2.2, Y1.1
- new net: C1.1, Y1.3
- new net: C3.2, U3.2 (VIN)
- new net: U2.1 (IOVDD), U2.10 (IOVDD), U2.22 (IOVDD), U2.33 (IOVDD), U2.42 (IOVDD), U2.49 (IOVDD)
- new net: U2.23 (DVDD), U2.50 (DVDD)
- new net +3.3V: C4.1, C5.2, U3.3 (VOUT), U4.8 (VCC)
- new net CLK: U2.52 (QSPI_SCLK), U4.6 (CLK)
- new net GND: C1.2, C2.1, C3.1, C4.2, C5.1, U3.1 (GND), U4.4 (GND), Y1.2, Y1.4
- new net IO0: U2.53 (QSPI_SD0), U4.5 (DI(IO0))
- new net IO1: U2.55 (QSPI_SD1), U4.2 (DO(IO1))
- new net IO2: U2.54 (QSPI_SD2), U4.3 (IO2)
- new net IO3: U2.51 (QSPI_SD3), U4.7 (IO3)
- new net ~{CS}: U2.56 (QSPI_SS), U4.1 (~{CS})
Other:
- note added: "X322512MSB4SI"

Commit message: updated files
Parts:
- U4: value W25Q32JVSS -> W25Q128
Changed lines of the file:
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@@
       (effects (font (size 1.27 1.27)) (justify left))
     )
-    (property "Value" "W25Q32JVSS" (id 1) (at 296.6594 149.86 0)
+    (property "Value" "W25Q128" (id 1) (at 296.6594 149.86 0)
       (effects (font (size 1.27 1.27)) (justify left))
     )
@@
     )
     (path "/758315a0-9b35-4bbd-943c-2b2f72fcca0b"
-      (reference "U4") (unit 1) (value "W25Q32JVSS") (footprint "Package_SO:SOIC-8_5.23x5.23mm_P1.27mm")
+      (reference "U4") (unit 1) (value "W25Q128") (footprint "Package_SO:SOIC-8_5.23x5.23mm_P1.27mm")
     )
     (path "/27be479a-ca38-4d90-b633-9076538762ca"

Commit message: updated files
Parts:
- added C? (x4): 10uF, Capacitor_SMD:C_0402_1005Metric, symbol Device:C_Small
Connections:
- net GND: now also C?.1, C?.1, C?.1, C?.1
- net at U2.1 (IOVDD), U2.10 (IOVDD), U2.22 (IOVDD)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: now also U2.43 (ADC_AVDD), U2.44 (VREG_IN), U2.48 (USB_VDD), C?.2, C?.2, C?.2
- net at U2.23 (DVDD), U2.50 (DVDD): now also U2.45 (VREG_VOUT), C?.2
Other:
- moved on the sheet: J1, J2, J3, J4

Commit message: updated files
Parts:
- removed C? (x2): 10uF, Capacitor_SMD:C_0402_1005Metric, symbol Device:C_Small
- removed J1, J2, J3, J4: Conn_01x09, Connector_PinHeader_1.27mm:PinHeader_1x09_P1.27mm_Vertical, symbol Connector_Generic:Conn_01x09
- removed U4: W25Q128, Package_SO:SOIC-8_5.23x5.23mm_P1.27mm, symbol Memory_Flash:W25Q32JVSS
- added C10, C11, C12, C13, C7, C8: 10uF, Capacitor_SMD:C_0402_1005Metric, symbol Device:C_Small
- added R1: 1K, Resistor_SMD:R_0402_1005Metric, symbol Device:R
- added R2, R3: 10K, Resistor_SMD:R_0402_1005Metric, symbol Device:R
- added R4: 22R, Resistor_SMD:R_0402_1005Metric, symbol Device:R
- added R5: 27R, Resistor_SMD:R_0402_1005Metric, symbol Device:R
- added SW1: RST, Button_Switch_SMD:SW_SPST_B3U-1000P, symbol Switch:SW_SPST
- added SW2: BOOTSEL, Button_Switch_SMD:SW_SPST_B3U-1000P, symbol Switch:SW_SPST
- added U6: W25Q64JVXGIQ_TR, 25Q64:W25Q64JVXGIQ TR, symbol 25Q64:W25Q64JVXGIQ_TR
- gave numbers to parts that had none: 2
Connections:
- net CLK: now also U6.6 (CLK)
- net GND: now also C5.2, U1.4 (GND1), U2.19 (TESTEN), U2.57 (GND), C10.1, C11.1, C12.1, C13.1, C7.1, C8.1, SW1.1 (A), SW2.1 (A), U6.4 (GND), U6.9 (EP); no longer C5.1
- net IO0: now also U6.5 (DI)
- net IO1: now also U6.2 (DO)
- net IO2: now also U6.3 (~{WP})
- net IO3: now also U6.7 (~{RST})
- net ~{CS}: now also R1.2, SW2.2 (B), U6.1 (~{CS})
- net at C2.2, Y1.1: now also U2.20 (XIN)
- net at C1.1, Y1.3: now also U2.21 (XOUT)
- net +3V3: now reaches C9.2, U2.1 (IOVDD), U2.10 (IOVDD), U2.22 (IOVDD), U2.33 (IOVDD), U2.42 (IOVDD), U2.43 (ADC_AVDD), U2.44 (VREG_IN), U2.48 (USB_VDD), U2.49 (IOVDD)
- net +3V3: now also C4.1, C5.1, U1.1 (VDD1), U3.3 (VOUT), C10.2, C11.2, C12.2, C13.2, R2.1, U6.8 (VCC)
- net +1V1: now reaches C6.2, U2.23 (DVDD), U2.45 (VREG_VOUT), U2.50 (DVDD)
- net +1V1: now also C7.2, C8.2
- net VCC: now reaches C3.2, U3.2 (VIN)
- net GPIO8: now reaches U2.11 (GPIO8)
- net GPIO9: now reaches U2.12 (GPIO9)
- net GPIO10: now reaches U2.13 (GPIO10)
- net GPIO11: now reaches U2.14 (GPIO11)
- net GPIO12: now reaches U2.15 (GPIO12)
- net GPIO13: now reaches U2.16 (GPIO13)
- net GPIO14: now reaches U2.17 (GPIO14)
- net GPIO15: now reaches U2.18 (GPIO15)
- net GPIO0: now reaches U2.2 (GPIO0)
- net RST: now reaches U2.26 (RUN)
- net RST: now also R3.2, SW1.2 (B)
- net GPIO16: now reaches U2.27 (GPIO16)
- net GPIO17: now reaches U2.28 (GPIO17)
- net GPIO18: now reaches U2.29 (GPIO18)
- net GPIO1: now reaches U2.3 (GPIO1)
- net GPIO19: now reaches U2.30 (GPIO19)
- net GPIO20: now reaches U2.31 (GPIO20)
- net GPIO21: now reaches U2.32 (GPIO21)
- net GPIO22: now reaches U2.34 (GPIO22)
- net GPIO23: now reaches U2.35 (GPIO23)
- net GPIO24: now reaches U2.36 (GPIO24)
- net GPIO25: now reaches U2.37 (GPIO25)
- net GPIO26: now reaches U2.38 (GPIO26_ADC0)
- net GPIO27: now reaches U2.39 (GPIO27_ADC1)
- net GPIO2: now reaches U2.4 (GPIO2)
- net GPIO28: now reaches U2.40 (GPIO28_ADC2)
- net GPIO29: now reaches U2.41 (GPIO29_ADC3)
- net at U2.46 (USB_DM): now also R4.2
- net at U2.47 (USB_DP): now also R5.2
- net GPIO3: now reaches U2.5 (GPIO3)
- net GPIO4: now reaches U2.6 (GPIO4)
- net GPIO5: now reaches U2.7 (GPIO5)
- net GPIO6: now reaches U2.8 (GPIO6)
- net GPIO7: now reaches U2.9 (GPIO7)
- net ISO_GND: now reaches U1.5 (GND2)
- net ISO_VO: now reaches U1.6 (VOB)
- net ISO_VIN: now reaches U1.7 (VIA)
- net ISO_VCC: now reaches U1.8 (VDD2)
- removed net +3.3V: C4.1, C5.2, U3.3 (VOUT)
- new net: R1.1, R2.2, R3.1
Other:
- moved on the sheet: C1, C2, C3, C4, C5, C6, C9, U1, U3, Y1

Commit message: updated files
Parts:
- added J1, J2, J3, J4: IO, Connector_PinHeader_2.00mm:PinHeader_1x10_P2.00mm_Vertical, symbol Connector_Generic:Conn_01x10
Connections:
- net +3V3: now also R3.1
- net GND: now also J4.1 (Pin_1)
- net VCC: now also J4.2 (Pin_2)
- net at R1.1, R2.2: no longer R3.1
Other:
- moved on the sheet: R2

Commit message: updated files
Connections:
- net SWCLK: now reaches U2.24 (SWCLK)
- net SWD: now reaches U2.25 (SWD)
Changed lines of the file:
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@@
+    (stroke (width 0) (type default) (color 0 0 0 0))
+  )
+  (wire (pts (xy 158.75 177.8) (xy 166.37 177.8))
     (stroke (width 0) (type default) (color 0 0 0 0))
   )
@@
     (stroke (width 0) (type default) (color 0 0 0 0))
   )
+  (wire (pts (xy 158.75 175.26) (xy 166.37 175.26))
+    (stroke (width 0) (type default) (color 0 0 0 0))
+  )
   (text "X322512MSB4SI" (at 93.98 203.2 0)
     (effects (font (size 1.27 1.27)) (justify left bottom))
@@
     (effects (font (size 1.27 1.27)) (justify right bottom))
   )
+  (label "SWCLK" (at 158.75 175.26 0)
+    (effects (font (size 1.27 1.27)) (justify left bottom))
+  )
   (label "GPIO29" (at 226.06 185.42 180)
     (effects (font (size 1.27 1.27)) (justify right bottom))
@@
     (effects (font (size 1.27 1.27)) (justify right bottom))
   )
+  (label "SWD" (at 158.75 177.8 0)
+    (effects (font (size 1.27 1.27)) (justify left bottom))
+  )
   (label "GPIO9" (at 226.06 132.08 180)

Commit message: updated files
Connections:
- net GND: now also J3.2 (Pin_2)
- net GPIO0: now also J4.10 (Pin_10)
- net GPIO1: now also J4.9 (Pin_9)
- net GPIO10: now also J3.8 (Pin_8)
- net GPIO11: now also J3.7 (Pin_7)
- net GPIO12: now also J3.6 (Pin_6)
- net GPIO13: now also J3.5 (Pin_5)
- net GPIO14: now also J3.4 (Pin_4)
- net GPIO15: now also J3.3 (Pin_3)
- net GPIO18: now also U1.3 (VIB)
- net GPIO19: now also U1.2 (VOA)
- net GPIO2: now also J4.8 (Pin_8)
- net GPIO3: now also J4.7 (Pin_7)
- net GPIO4: now also J4.6 (Pin_6)
- net GPIO5: now also J4.5 (Pin_5)
- net GPIO6: now also J4.4 (Pin_4)
- net GPIO7: now also J4.3 (Pin_3)
- net GPIO8: now also J3.10 (Pin_10)
- net GPIO9: now also J3.9 (Pin_9)
- net RST: now also J3.1 (Pin_1)
Other:
- moved on the sheet: J1, J2, J3

Commit message: updated files
Connections:
- net GPIO22: now also J1.9 (Pin_9)
- net GPIO23: now also J1.8 (Pin_8)
- net GPIO24: now also J1.7 (Pin_7)
- net GPIO25: now also J1.6 (Pin_6)
- net GPIO26: now also J1.5 (Pin_5)
- net GPIO27: now also J1.4 (Pin_4)
- net GPIO28: now also J1.3 (Pin_3)
- net GPIO29: now also J1.2 (Pin_2)
- net ISO_GND: now also J2.4 (Pin_4)
- net ISO_VCC: now also J2.1 (Pin_1)
- net ISO_VIN: now also J2.2 (Pin_2)
- net ISO_VO: now also J2.3 (Pin_3)
- net ~{CS}: now also J1.1 (Pin_1)
Other:
- moved on the sheet: J1, J2
